Commit message: implemented improved wheel pid

File: hardware/wheel-can-hardware/urdf/rover_wheels.ros2_control.xacro (robot description, xacro)
@@ -17,5 +17,7 @@
 -->
 <robot xmlns:xacro="http://www.ros.org/wiki/xacro">
-  <xacro:macro name="rover_wheels_ros2_control" params="name:='RoverWheels' can_interface:='can0'">
+  <xacro:macro name="rover_wheels_ros2_control" params="name:='RoverWheels' can_interface:='can0' traction_mode:='assist' control_mode:='velocity'">
+    <!-- velocity mode -> velocity command interface; current mode -> effort. -->
+    <xacro:property name="cmd_if" value="${'effort' if control_mode == 'current' else 'velocity'}"/>
     <ros2_control name="${name}" type="system">
       <hardware>
@@ -24,12 +26,25 @@
         <param name="send_heartbeat_on_activate">true</param>
         <param name="heartbeat_motor_mask">0x7E</param>
-        <!-- anti_slip_mode: off | clamp | pid | current_pid -->
+        <!-- control_mode: velocity (RPM, with traction/anti-slip) | current
+             (amperes, open loop). max_current_a clamps the current setpoint. -->
+        <param name="control_mode">${control_mode}</param>
+        <param name="max_current_a">25.0</param>
+        <!-- Traction (Step A): redistribute each side's RPM toward gripping
+             wheels before anti-slip. traction_mode: off | assist | aggressive -->
+        <param name="traction_mode">${traction_mode}</param>
+        <param name="traction_slip_free_threshold">0.4</param>
+        <param name="traction_slip_stall_threshold">-0.3</param>
+        <param name="traction_min_weight">0.1</param>
+        <param name="traction_low_load_a">2.0</param>
+        <param name="traction_weight_k">0.5</param>
+        <!-- Anti-slip (Step B), setpoint is the post-traction target_rpm.
+             anti_slip_mode: off | clamp | pid | current_pid -->
         <param name="anti_slip_mode">pid</param>
         <param name="slip_threshold">0.30</param>
         <param name="slip_kp">0.10</param>
         <param name="max_slip_correction">0.50</param>
-        <param name="feedback_freshness_ms">50.0</param>
-        <!-- Only consulted by current_pid mode -->
-        <param name="stall_current_a">30.0</param>
+        <param name="feedback_freshness_ms">100.0</param>
+        <!-- stall guard: shared by traction motor-protect and current_pid -->
+        <param name="stall_current_a">20.0</param>
         <param name="stall_relief_factor">0.50</param>
       </hardware>
@@ -39,5 +54,5 @@
         <param name="direction">-1.0</param>
         <param name="gear_ratio">1.0</param>
-        <command_interface name="velocity"/>
+        <command_interface name="${cmd_if}"/>
         <state_interface name="velocity"/>
         <state_interface name="position"/>
@@ -48,5 +63,5 @@
         <param name="direction">-1.0</param>
         <param name="gear_ratio">1.0</param>
-        <command_interface name="velocity"/>
+        <command_interface name="${cmd_if}"/>
         <state_interface name="velocity"/>
         <state_interface name="position"/>
@@ -57,5 +72,5 @@
         <param name="direction">-1.0</param>
         <param name="gear_ratio">1.0</param>
-        <command_interface name="velocity"/>
+        <command_interface name="${cmd_if}"/>
         <state_interface name="velocity"/>
         <state_interface name="position"/>
@@ -66,5 +81,5 @@
         <param name="direction">1.0</param>
         <param name="gear_ratio">1.0</param>
-        <command_interface name="velocity"/>
+        <command_interface name="${cmd_if}"/>
         <state_interface name="velocity"/>
         <state_interface name="position"/>
@@ -75,5 +90,5 @@
         <param name="direction">1.0</param>
         <param name="gear_ratio">1.0</param>
-        <command_interface name="velocity"/>
+        <command_interface name="${cmd_if}"/>
         <state_interface name="velocity"/>
         <state_interface name="position"/>
@@ -84,5 +99,5 @@
         <param name="direction">1.0</param>
         <param name="gear_ratio">1.0</param>
-        <command_interface name="velocity"/>
+        <command_interface name="${cmd_if}"/>
         <state_interface name="velocity"/>
         <state_interface name="position"/>

File: hardware/wheel-can-hardware/urdf/test_rover_wheels.urdf.xacro (robot description, xacro)
@@ -7,4 +7,6 @@
 <robot xmlns:xacro="http://www.ros.org/wiki/xacro" name="test_rover_wheels">
   <xacro:arg name="can_interface" default="can0"/>
+  <xacro:arg name="traction_mode" default="assist"/>
+  <xacro:arg name="control_mode" default="velocity"/>
   <!-- Minimal kinematic tree: ros2_control joint names must exist in URDF. -->
   <xacro:macro name="bench_wheel" params="joint_name link_name xyz:='0 0 0'">
@@ -35,4 +37,4 @@
   <xacro:bench_wheel joint_name="wheel_left_rear"    link_name="wheel_left_rear_link"    xyz="-0.4 0.6 0"/>
   <xacro:include filename="$(find wheel_can_hardware)/urdf/rover_wheels.ros2_control.xacro"/>
-  <xacro:rover_wheels_ros2_control name="RoverWheels" can_interface="$(arg can_interface)"/>
+  <xacro:rover_wheels_ros2_control name="RoverWheels" can_interface="$(arg can_interface)" traction_mode="$(arg traction_mode)" control_mode="$(arg control_mode)"/>
 </robot>
