Commit message: added wheel telem and launch options

File: hardware/wheel-can-hardware/urdf/rover_arm_and_wheels.urdf.xacro (robot description, xacro)
@@ -57,8 +57,8 @@
   <xacro:wheel_link joint_name="wheel_left_rear"   link_name="wheel_left_rear_link"   xyz="-0.4  0.6 0"/>
   <!-- Arm ros2_control hardware block (ArmCanInterface). -->
-  <xacro:include filename="$(find rover_arm_moveit_config)/config/rover_arm.ros2_control.xacro"/>
-  <xacro:rover_arm_ros2_control
+  <xacro:include filename="$(find arm_can_hardware)/urdf/rover_arm_can.ros2_control.xacro"/>
+  <xacro:rover_arm_can_ros2_control
       name="RoverArm"
-      initial_positions_file="$(arg initial_positions_file)"/>
+      can_interface="$(arg can_interface)"/>
   <!-- Wheel ros2_control hardware block (WheelCanInterface). -->
   <xacro:include filename="$(find wheel_can_hardware)/urdf/rover_wheels.ros2_control.xacro"/>

File: hardware/wheel-can-hardware/urdf/rover_wheels.ros2_control.xacro (robot description, xacro)
@@ -17,5 +17,5 @@
 -->
 <robot xmlns:xacro="http://www.ros.org/wiki/xacro">
-  <xacro:macro name="rover_wheels_ros2_control" params="name:='RoverWheels' can_interface:='can0' traction_mode:='assist' control_mode:='velocity'">
+  <xacro:macro name="rover_wheels_ros2_control" params="name:='RoverWheels' can_interface:='can0' traction_mode:='assist' control_mode:='velocity' log_telemetry:='false' print_period_ms:='1000'">
     <!-- velocity mode -> velocity command interface; current mode -> effort. -->
     <xacro:property name="cmd_if" value="${'effort' if control_mode == 'current' else 'velocity'}"/>
@@ -45,4 +45,7 @@
         <param name="max_slip_correction">0.50</param>
         <param name="feedback_freshness_ms">100.0</param>
+        <!-- Periodic SPARK telemetry table (wheel_bench_node layout). -->
+        <param name="log_telemetry">${log_telemetry}</param>
+        <param name="print_period_ms">${print_period_ms}</param>
         <!-- stall guard: shared by traction motor-protect and current_pid -->
         <param name="stall_current_a">20.0</param>

File: hardware/wheel-can-hardware/urdf/test_rover_wheels.urdf.xacro (robot description, xacro)
@@ -9,4 +9,6 @@
   <xacro:arg name="traction_mode" default="assist"/>
   <xacro:arg name="control_mode" default="velocity"/>
+  <xacro:arg name="log_telemetry" default="true"/>
+  <xacro:arg name="print_period_ms" default="1000"/>
   <!-- Minimal kinematic tree: ros2_control joint names must exist in URDF. -->
   <xacro:macro name="bench_wheel" params="joint_name link_name xyz:='0 0 0'">
@@ -37,4 +39,4 @@
   <xacro:bench_wheel joint_name="wheel_left_rear"    link_name="wheel_left_rear_link"    xyz="-0.4 0.6 0"/>
   <xacro:include filename="$(find wheel_can_hardware)/urdf/rover_wheels.ros2_control.xacro"/>
-  <xacro:rover_wheels_ros2_control name="RoverWheels" can_interface="$(arg can_interface)" traction_mode="$(arg traction_mode)" control_mode="$(arg control_mode)"/>
+  <xacro:rover_wheels_ros2_control name="RoverWheels" can_interface="$(arg can_interface)" traction_mode="$(arg traction_mode)" control_mode="$(arg control_mode)" log_telemetry="$(arg log_telemetry)" print_period_ms="$(arg print_period_ms)"/>
 </robot>
