Commit message: switched arm MoveitConfig to CAN hardware

File: inverse-kinematics/rover_arm_description/urdf/arm.xacro (robot description, xacro)
@@ -123,5 +123,5 @@
         <axis xyz="1 0 0"/>
     </joint>
-   <joint name="joint4" type="fixed">
+   <joint name="joint4" type="continuous">
         <parent link="bicep_gearbox_link"/>
         <child link="forearm_tube_link"/>
@@ -135,8 +135,9 @@
         <axis xyz=" 1 0 0"/>
     </joint>
-    <joint name="joint6" type="fixed">
+    <joint name="joint6" type="continuous">
         <parent link="bracket_connection_link"/>
         <child link="gripper_base_link"/>
         <origin xyz="-0.026225 0 0.070075" rpy="0 0 0"/>
+        <axis xyz=" 0 0 1"/>
     </joint>
 </robot>

File: inverse-kinematics/rover_arm_moveit_config/config/rover_arm.urdf.xacro (robot description, xacro)
@@ -2,8 +2,23 @@
 <robot xmlns:xacro="http://www.ros.org/wiki/xacro" name="rover_arm">
     <xacro:arg name="initial_positions_file" default="initial_positions.yaml" />
+    <xacro:arg name="can_interface" default="can0" />
+    <!-- hardware_backend: "can" (default, ArmCanInterface over CAN),
+         "fake" (mock_components for MoveIt planning demos), or
+         "serial" (legacy arm_interface/ArmInterface on /dev/ttyUSB0 + /dev/ttyTHS1). -->
+    <xacro:arg name="hardware_backend" default="can" />
     <!-- Import rover_arm urdf file -->
     <xacro:include filename="$(find rover_arm_description)/urdf/arm.urdf.xacro" />
-    <!-- Import control_xacro -->
-    <xacro:include filename="rover_arm.ros2_control.xacro" />
-    <xacro:rover_arm_ros2_control name="FakeSystem" initial_positions_file="$(arg initial_positions_file)"/>
+    <xacro:property name="hardware_backend" value="$(arg hardware_backend)" />
+    <xacro:if value="${hardware_backend == 'can'}">
+        <xacro:include filename="$(find arm_can_hardware)/urdf/rover_arm_can.ros2_control.xacro" />
+        <xacro:rover_arm_can_ros2_control name="RoverArm" can_interface="$(arg can_interface)" />
+    </xacro:if>
+    <xacro:if value="${hardware_backend == 'fake'}">
+        <xacro:include filename="rover_arm_fake.ros2_control.xacro" />
+        <xacro:rover_arm_fake_ros2_control name="FakeRoverArm" initial_positions_file="$(arg initial_positions_file)" />
+    </xacro:if>
+    <xacro:if value="${hardware_backend == 'serial'}">
+        <xacro:include filename="rover_arm_serial.ros2_control.xacro" />
+        <xacro:rover_arm_ros2_control name="FakeSystem" initial_positions_file="$(arg initial_positions_file)" />
+    </xacro:if>
 </robot>

File: inverse-kinematics/rover_arm_moveit_config/config/rover_arm_serial.ros2_control.xacro (robot description, xacro)
@@ -1,3 +1,10 @@
 <?xml version="1.0"?>
+<!--
+  LEGACY serial ros2_control block for the rover arm (arm_interface/ArmInterface):
+  ABSENC encoders on /dev/ttyUSB0 and motor commands on /dev/ttyTHS1.
+  Kept for reference only. The arm has moved to CAN; production uses
+  arm_can_hardware/ArmCanInterface via rover_arm_can.ros2_control.xacro.
+  Select this path with hardware_backend:=serial in rover_arm.urdf.xacro.
+-->
 <robot xmlns:xacro="http://www.ros.org/wiki/xacro">
     <xacro:macro name="rover_arm_ros2_control" params="name initial_positions_file">
